Commit message: fase 1 terminada comienzo fase 2

File: practica_1/URDFs/barrera.urdf (robot description, URDF)
Before this commit: robot barrera, 2 links, 1 joints
Links:
- link barrier_link: geometry collision box size=2.5 0.1 0.1; visual box size=2.5 0.1 0.1
Joints:
- joint barrier_joint: origin xyz=0.0 0.0 0.25 rpy=0.0 0.0 0.0 -> xyz=0.0 0.0 0.15 rpy=0.0 0.0 0.0

Commit message: fase 3 terminada

File: practica_1/URDFs/barrera.urdf (robot description, URDF)
Before this commit: robot barrera, 2 links, 1 joints
Links:
- link barrier_link: mass None -> 5.0

File: practica_1/URDFs/rampa.urdf (robot description, URDF)
Before this commit: robot rampa, 3 links, 2 joints
Links:
- link base_link: mass 100.0 -> None
- link downwards_link: mass 40.0 -> None
- link upwards_link: mass 40.0 -> None
