Commit message: puntos de aproximacion hechos

File: practica_2/rover_scara/urdf/rover_scara.urdf (robot description, URDF)
Before this commit: robot rover_scara, 14 links, 13 joints
Joints:
- joint Seg1_link_joint: limit lower=-3.00000 upper=3.00000 effort=0.00000 velocity=0.00000 -> lower=-6.00000 upper=6.00000 effort=0.00000 velocity=0.00000

Commit message: coger cubo hecho

File: practica_2/rover_scara/urdf/rover_scara.urdf (robot description, URDF)
Before this commit: robot rover_scara, 14 links, 13 joints
Joints:
- joint Seg1_link_joint: limit lower=-6.00000 upper=6.00000 effort=0.00000 velocity=0.00000 -> lower=-3.00000 upper=3.00000 effort=0.00000 velocity=0.00000
