Commit message: practica 3 empezada

File: modelado-ws/src/roverto_description/robots/roverto.urdf.xacro (robot description, xacro)
@@ -1,36 +1,26 @@
-<robot name="robot" xmlns:xacro="http://wiki.ros.org/xacro">
-<!-- includes -->
-<xacro:include filename="$(find roverto_description)/urdf/base/robot_base.urdf.xacro"/>
-<xacro:include filename="$(find roverto_description)/urdf/wheels/roverTo_wheel.urdf.xacro"/>
-<xacro:include filename="$(find roverto_description)/urdf/arm/scara.urdf.xacro"/>
-<xacro:include filename="$(find roverto_description)/urdf/arm/gripper.urdf.xacro"/>
-<xacro:include filename="$(find roverto_description)/urdf/sensors/camera.urdf.xacro"/>
-<xacro:include filename="$(find roverto_description)/urdf/sensors/imu_sensor.urdf.xacro"/>
-<!-- Robot Parts -->
-<!-- Base -->
-<xacro:base parent="base_footprint"/>
-<!-- Wheels -->
-<xacro:wheels parent="base_link"/>
-<!-- Arm -->
-<xacro:scara parent="base_link"/>
-<xacro:fingers parent="Seg4_link"/>
-<!-- sensores -->
-<xacro:base_camera prefix="base" parent="base_link" xyz="0.0 -1.8 0.2" rpy="1.57 3.14 0.0"/>
-<xacro:base_camera prefix="gripper" parent="Seg4_link" xyz="0.0 0.0 0.0" rpy="0.0 3.14 0.0"/>
-<xacro:imu parent="base_link"/>
-<!-- <xacro:sensor_camera node_name="front_camera" node_namespace="$(arg robot_ns)" frame_prefix="$(arg prefix)front_camera_" parent="$(arg prefix)base_link">
-<origin xyz="0.0 1.4 0.5" rpy="0 0 ${PI/2}"/>
-</xacro:sensor_camera> -->
-<!-- xacro:sensor_camera node_name="arm_camera" node_namespace="$(arg robot_ns)" frame_prefix="$(arg prefix)arm_camera_" parent="$(arg prefix)base_effector_arm_link" >
-        <origin xyz="0.0 0.0 -0.01" rpy="0 3.141592 0"/>
-    </xacro:sensor_camera
- <xacro:sensor_imu ns="$(arg robot_ns)" prefix="$(arg prefix)imu_" parent="$(arg prefix)base_link">
-        <origin xyz="0.0 0.0 0.0" rpy="0 0 0"/>
-    </xacro:sensor_imu>
- Gazebo ROS control plugins
-<xacro:include filename="$(find msr_robot)/urdf/ros2_control.urdf.xacro"/>
- <xacro:arg name="config_controllers" default="$(find gz_ros2_control_demos)/config/diff_drive_controller.yaml"/>
-<xacro:arg name="config_controllers" default="$(find msr_robot)/config/rover_controllers.yaml"/>
-<xacro:arg name="update_rate" default="100"/>
-<xacro:ros2_control/> -->
+<robot name="roverto" xmlns:xacro="http://wiki.ros.org/xacro">
+    <!-- includes -->
+    <xacro:include filename="$(find roverto_description)/urdf/base/robot_base.urdf.xacro"/>
+    <xacro:include filename="$(find roverto_description)/urdf/wheels/roverTo_wheel.urdf.xacro"/>
+    <xacro:include filename="$(find roverto_description)/urdf/arm/scara.urdf.xacro"/>
+    <xacro:include filename="$(find roverto_description)/urdf/arm/gripper.urdf.xacro"/>
+    <xacro:include filename="$(find roverto_description)/urdf/sensors/camera.urdf.xacro"/>
+    <xacro:include filename="$(find roverto_description)/urdf/sensors/imu_sensor.urdf.xacro"/>
+    <!-- Robot Parts -->
+    <!-- Base -->
+    <xacro:base parent="base_footprint"/>
+    <!-- Wheels -->
+    <xacro:wheels parent="base_link"/>
+    <!-- Arm -->
+    <xacro:scara parent="base_link"/>
+    <xacro:fingers parent="Seg4_link"/>
+    <!-- sensores -->
+    <xacro:base_camera prefix="base" parent="base_link" xyz="0.0 -1.8 0.2" rpy="1.57 3.14 0.0"/>
+    <xacro:base_camera prefix="gripper" parent="Seg4_link" xyz="0.0 0.0 0.0" rpy="0.0 3.14 0.0"/>
+    <xacro:imu parent="base_link"/>
+    <!-- Gazebo ROS control plugins -->
+    <xacro:include filename="$(find roverto_description)/urdf/ros2_control.urdf.xacro"/>
+    <xacro:arg name="config_controllers" default="$(find roverto_description)/config/rover_controllers.yaml"/>
+    <xacro:arg name="update_rate" default="20"/>
+    <xacro:ros2_control/>
 </robot>

File: modelado-ws/src/roverto_description/urdf/arm/gripper.urdf.xacro (robot description, xacro)
@@ -4,5 +4,5 @@
   <xacro:macro name="finger" params="prefix parent xyz rpy">
     <joint name="${prefix}_joint" type="prismatic">
-      <limit lower="0.00000" upper="0.25000" effort="0.00000" velocity="0.00000"/>
+      <limit lower="0.00000" upper="0.25000" effort="1000" velocity="100.0"/>
       <origin rpy="${rpy}" xyz="${xyz}"/>
       <parent link="Seg4_link"/>

File: modelado-ws/src/roverto_description/urdf/arm/scara.urdf.xacro (robot description, xacro)
@@ -10,5 +10,5 @@
     </joint>
     <joint name="Seg1_link_joint" type="revolute">
-      <limit lower="-3.00000" upper="3.00000" effort="0.00000" velocity="0.00000"/>
+      <limit lower="-3.00000" upper="3.00000" effort="1000.0" velocity="100.0"/>
       <origin rpy="0.00000 0.00000 0.00000" xyz="0.00000 0.02000 1.60000"/>
       <parent link="base_brazo_link"/>
@@ -17,5 +17,5 @@
     </joint>
     <joint name="Seg2_link_joint" type="revolute">
-      <limit lower="-0.70000" upper="4.00000" effort="0.00000" velocity="0.00000"/>
+      <limit lower="-0.70000" upper="4.00000" effort="1000.0" velocity="100.0"/>
       <origin rpy="0.00000 0.00000 0.00000" xyz="-0.00000 1.48000 -0.17250"/>
       <parent link="Seg1_link"/>
@@ -24,5 +24,5 @@
     </joint>
     <joint name="Seg3_link_joint" type="prismatic">
-      <limit lower="-2.50000" upper="0.00000" effort="0.00000" velocity="0.00000"/>
+      <limit lower="-2.50000" upper="0.00000" effort="1000.0" velocity="100.0"/>
       <origin rpy="0.00000 0.00000 0.00000" xyz="1.80000 -0.00000 1.17250"/>
       <parent link="Seg2_link"/>
@@ -31,5 +31,5 @@
     </joint>
     <joint name="Seg4_link_joint" type="continuous">
-      <limit lower="0" upper="0" effort="0.00000" velocity="0.00000"/>
+      <limit lower="0" upper="0" effort="1000.0" velocity="100.0"/>
       <origin rpy="0.00000 0.00000 0.00000" xyz="-0.00000 -0.00000 -1.60000"/>
       <parent link="Seg3_link"/>

File: modelado-ws/src/roverto_description/urdf/sensors/camera.urdf.xacro (robot description, xacro)
@@ -3,5 +3,4 @@
 <robot name="base_camera" xmlns:xacro="http://www.ros.org/wiki/xacro">
     <xacro:macro name="base_camera" params="prefix parent xyz rpy">
-<!-- CORREGIR ROTACION JOINTS -->
     <!-- Joints -->
     <joint name="${prefix}_camera_joint" type="fixed">
@@ -31,4 +30,29 @@
     <link name="${prefix}_camera_frame"/>
     <link name="${prefix}_camera_optical_frame"/>
+    <gazebo reference="${prefix}_camera_frame">
+      <sensor name="${prefix}_sensor" type="camera">
+        <visualize>true</visualize>
+        <update_rate>30</update_rate>
+        <topic>/${prefix}/image</topic>
+        <camera>
+          <horizontal_fov>${radians(float(80))}</horizontal_fov>
+          <image>
+            <width>1280</width>
+            <height>720</height>
+            <format>R8G8B8</format>
+          </image>
+          <clip>
+            <near>0.10</near>
+            <far>15.0</far>
+          </clip>
+          <noise>
+            <type>gaussian</type>
+            <mean>0.0</mean>
+            <stddev>0.007</stddev>
+          </noise>
+          <optical_frame_id>${prefix}_camera_frame</optical_frame_id>
+        </camera>
+      </sensor>
+    </gazebo>
     </xacro:macro>
 </robot>

File: modelado-ws/src/roverto_description/urdf/sensors/imu_sensor.urdf.xacro (robot description, xacro)
@@ -2,13 +2,20 @@
 <!-- created with Phobos 1.0.1 "Capricious Choutengan" -->
 <robot name="imu" xmlns:xacro="http://www.ros.org/wiki/xacro">
-    <xacro:macro name="imu" params="parent">
-    <!-- Joints -->
-    <joint name="imu_joint" type="fixed">
-      <origin rpy="0.00000 0.00000 0.00000" xyz="0.0 0.0 0.0"/>
-      <parent link="${parent}"/>
-      <child link="imu_link"/>
-    </joint>
-    <!-- Link -->
-    <link name="imu_link"/>
+    <xacro:macro name="imu" params="parent topic:='imu/data'">
+      <!-- Joints -->
+      <joint name="imu_joint" type="fixed">
+        <origin rpy="0.00000 0.00000 0.00000" xyz="0.0 0.0 0.0"/>
+        <parent link="${parent}"/>
+        <child link="imu_link"/>
+      </joint>
+      <!-- Link -->
+      <link name="imu_link"/>
+      <gazebo reference="imu_link">
+        <sensor name="imu_sensor" type="imu">
+          <always_on>1</always_on>
+          <update_rate>30</update_rate>
+          <topic>${topic}</topic>
+        </sensor>
+      </gazebo>
     </xacro:macro>
 </robot>

File: modelado-ws/src/roverto_description/urdf/wheels/roverTo_wheel.urdf.xacro (robot description, xacro)
@@ -3,25 +3,6 @@
 <robot name="base" xmlns:xacro="http://wiki.ros.org/xacro">
   <xacro:macro name="wheel" params="prefix parent xyz rpy">
-    <link name="${prefix}_link">
-      <collision name="${prefix}_collision">
-          <origin rpy="0.00000 0.00000 0.00000" xyz="0.00000 0.00000 0.00000"/>
-          <geometry>
-              <mesh filename="file://$(find roverto_description)/dae/Cilindro.005.dae" scale="0.30000 0.30000 0.10000"/>
-          </geometry>
-          </collision>
-          <inertial>
-              <inertia ixx="1.17477" ixy="0.00000" ixz="-0.00000" iyy="0.62554" iyz="-0.00000" izz="0.62554"/>
-              <origin rpy="0.00000 0.00000 0.00000" xyz="0.00000 0.00000 -0.01040"/>
-              <mass value="15.00000"/>
-          </inertial>
-          <visual name="${prefix}">
-              <origin rpy="0.00000 -0.00000 0.00000" xyz="0.00000 0.00000 0.00000"/>
-              <geometry>
-                  <mesh filename="file://$(find roverto_description)/dae/Cilindro.005.dae" scale="0.30000 0.30000 0.10000"/>
-              </geometry>
-          </visual>
-    </link>
     <joint name="${prefix}_wheel_joint" type="continuous">
-      <limit lower="0" upper="0" effort="0.00000" velocity="0.00000"/>
+      <limit lower="0" upper="0" effort="1000" velocity="100.0"/>
       <origin xyz="${xyz}" rpy="${rpy}"/>
       <parent link="${parent}"/>
@@ -29,4 +10,47 @@
       <axis xyz="0.00000 0.00000 1.00000"/>
     </joint>
+    <link name="${prefix}_link">
+      <collision name="${prefix}_collision">
+        <origin rpy="0.00000 0.00000 0.00000" xyz="0.00000 0.00000 0.00000"/>
+        <geometry>
+          <mesh filename="file://$(find roverto_description)/dae/Cilindro.005.dae" scale="0.30000 0.30000 0.10000"/>
+        </geometry>
+        <surface>
+          <friction>
+            <ode>
+              <mu>1.000000</mu>
+              <mu2>1.000000</mu2>
+              <fdir1>0.000000 0.000000 1.000000</fdir1>
+              <slip1>0.500000</slip1>
+              <slip2>0.500000</slip2>
+            </ode>
+          </friction>
+        </surface>
+      </collision>
+      <inertial>
+        <inertia ixx="1.17477" ixy="0.00000" ixz="-0.00000" iyy="0.62554" iyz="-0.00000" izz="0.62554"/>
+        <origin rpy="0.00000 0.00000 0.00000" xyz="0.00000 0.00000 -0.01040"/>
+        <mass value="15.00000"/>
+      </inertial>
+      <visual name="${prefix}">
+        <origin rpy="0.00000 -0.00000 0.00000" xyz="0.00000 0.00000 0.00000"/>
+        <geometry>
+          <mesh filename="file://$(find roverto_description)/dae/Cilindro.005.dae" scale="0.30000 0.30000 0.10000"/>
+        </geometry>
+      </visual>
+    </link>
+    <transmission name="${prefix}_wheel_joint_trans">
+      <type>transmission_interface/SimpleTransmission</type>
+      <joint name="${prefix}_wheel_joint">
+        <hardwareInterface>hardware_interface/VelocityJointInterface</hardwareInterface>
+      </joint>
+      <actuator name="${prefix}wheel_joint_motor">
+        <mechanicalReduction>1.0</mechanicalReduction>
+      </actuator>
+    </transmission>
+    <gazebo reference="${prefix}wheel_link">
+      <mu1>5</mu1>
+      <mu2>5</mu2>
+    </gazebo>
   </xacro:macro>
   <xacro:macro name="wheels" params="parent">
